File: circuit-diagram/circuit-diagram.kicad_sch (KiCad schematic)
At the start: 3 parts, among them M1 Motor_DC_ALT, U1 A3144

Commit message: Updated README and schematic
Parts:
- added D1: LED, symbol Device:LED
- added J1: UART Pins, symbol Connector:Conn_01x03_Pin
- added J2: DEBUG, symbol Connector:Conn_01x05_Pin
- added J3: MCU Power Input, symbol Connector:Conn_01x02_Pin
- added J4: Motor Power Input, symbol Connector:Conn_01x02_Pin
- added R2: 10k, symbol Device:R
- added R3: 470, symbol Device:R
- added SW1: RST, symbol Switch:SW_Push
- added SW2: SW_Push, symbol Switch:SW_Push
- added U2: A3144, Package_TO_SOT_SMD:SOT-23W, symbol Sensor_Magnetic:A1101ELHL
- added U3: VL53L0CXV0DH1, Sensor_Distance:ST_VL53L1x, symbol Sensor_Distance:VL53L0CXV0DH1
- R1: value R -> 10k
Connections:
- net +3V3: now also J2.5 (Pin_5), R2.1, U2.1 (VCC), U3.11 (AVDD)
- net +5V: now also J3.2 (Pin_2), J4.2 (Pin_2)
- net DBG_SWCLK: now also J2.4 (Pin_4)
- net DBG_SWDIO: now also J2.3 (Pin_3)
- net GND: now also J1.1 (Pin_1), J2.1 (Pin_1), J3.1 (Pin_1), J4.1 (Pin_1), R3.2, SW1.1, SW2.2, U2.3 (GND), U3.12 (GND), U3.3 (GND), U3.4 (GND), U3.6 (GND)
- net I2C0_SCL: now also U3.10 (SCL)
- net I2C0_SDA: now also U3.9 (SDA)
- net UART0_RX: now also J1.3 (Pin_3)
- net UART0_TX: now also J1.2 (Pin_2)
- net HALL_SENSOR renamed SPEED_HALL_SENSOR
- new net: D1.1 (K), R3.1
- new net DBG_RESET: J2.2 (Pin_2), SW1.2
- new net PUSH_BTN: SW2.1
- new net USER_LED: D1.2 (A)
- new net ZERO_HALL_SENSOR: R2.2, U2.2 (VOUT)
- no-connect marks 4 -> 8
Other:
- note added: "Connectors for debugging, power and UART output. Wiring here can be arbritary depending on how you want it For example, you can connect the motor and MCU power supplies together or make it possible to use a strong supply for the motor and a weaker one (e.g. a debug probe) just for the MCU."
- note added: "Sensors"
- note added: "Short Range Distance Sensor VL53L0X"
- note added: "User button and LED"
